File: ledcontroller.sch (KiCad schematic (older format))
At the start: 39 parts, among them J1 Barrel_Jack, J2 RGBW analog, J3 RGB addressable, J4 Conn_01x05_Male, Q1 DMN3404L, Q2 DMN3404L, Q3 DMN3404L, Q4 DMN3404L, Q5 DMN3404L, Q6 DMN3404L, Q7 DMN3404L, Q8 DMN3404L, U1 TPS54233, U2 ESP32-WROOM-32

Commit message: fixes #4 #3 #2
Parts:
- J4: value Conn_01x05_Male -> Conn_01x06_Male; footprint Connector_PinHeader_2.54mm:PinHeader_1x05_P2.54mm_Vertical -> Connector_PinHeader_2.54mm:PinHeader_1x06_P2.54mm_Vertical; symbol Connector:Conn_01x05_Male -> Connector:Conn_01x06_Male
Connections:
- net B1: now also U2.28 (IO17); no longer U2.8 (IO32)
- net G1: now also U2.27 (IO16); no longer U2.6 (IO34)
- net GND: now also J4.6 (Pin_6); no longer J4.5 (Pin_5)
- net R1: now also U2.30 (IO18); no longer U2.7 (IO35)
- net W1: now also U2.26 (IO4); no longer U2.9 (IO33)
- net EN: now reaches R6.2, U2.3 (EN)
- net EN: now also J4.5 (Pin_5)
Changed lines of the file:
@@
 Text Label 8000 2950 0    50   ~ 0
 W1
-Text Label 5350 6400 0    50   ~ 0
+Text Label 5350 5200 0    50   ~ 0
 G1
-Text Label 5350 6500 0    50   ~ 0
+Text Label 5350 5400 0    50   ~ 0
 R1
-Text Label 5350 6200 0    50   ~ 0
+Text Label 5350 5300 0    50   ~ 0
 B1
-Text Label 5350 6300 0    50   ~ 0
+Text Label 5350 4600 0    50   ~ 0
 W1
 Text Label 10000 6150 0    50   ~ 0
@@
 	9350 4450 10300 4450
 $Comp
-L Connector:Conn_01x05_Male J4
+L Connector:Conn_01x06_Male J4
 U 1 1 5E7462E3
 P 6500 4600
 F 0 "J4" H 6472 4624 50  0000 R CNN
-F 1 "Conn_01x05_Male" H 6472 4533 50  0000 R CNN
-F 2 "Connector_PinHeader_2.54mm:PinHeader_1x05_P2.54mm_Vertical" H 6500 4600 50  0001 C CNN
+F 1 "Conn_01x06_Male" H 6472 4533 50  0000 R CNN
+F 2 "Connector_PinHeader_2.54mm:PinHeader_1x06_P2.54mm_Vertical" H 6500 4600 50  0001 C CNN
 F 3 "~" H 6500 4600 50  0001 C CNN
 	1    6500 4600
@@
 L power:GND #PWR0131
 U 1 1 5E753E82
-P 6300 4800
-F 0 "#PWR0131" H 6300 4550 50  0001 C CNN
-F 1 "GND" H 6305 4627 50  0000 C CNN
-F 2 "" H 6300 4800 50  0001 C CNN
-F 3 "" H 6300 4800 50  0001 C CNN
-	1    6300 4800
+P 6300 4900
+F 0 "#PWR0131" H 6300 4650 50  0001 C CNN
+F 1 "GND" H 6305 4727 50  0000 C CNN
+F 2 "" H 6300 4900 50  0001 C CNN
+F 3 "" H 6300 4900 50  0001 C CNN
+	1    6300 4900
 	1    0    0    -1
 $EndComp
@@
 Wire Wire Line
 	5750 4700 6300 4700
+Connection ~ 4150 4200
+Text Label 4000 4200 0    50   ~ 0
+EN
+Text Label 6200 4800 0    50   ~ 0
+EN
+Wire Wire Line
+	6200 4800 6300 4800
+Wire Wire Line
+	4000 4200 4150 4200
 $EndSCHEMATC
